Commit message: fixed collision box clipping into ground, causing need for extreme force

File: src/my_rover/urdf/rover.urdf.xacro (robot description, xacro)
@@ -1,47 +1,40 @@
 <?xml version="1.0"?>
-<robot name="my_rover" xmlns:xacro="http://www.ros.org/wiki/xacro">
-  <!-- Include macros -->
+<robot name="rover" xmlns:xacro="http://ros.org/wiki/xacro">
+  <!-- Include wheel macro -->
   <xacro:include filename="$(find my_rover)/urdf/wheel_macro.xacro"/>
-  <xacro:include filename="$(find my_rover)/urdf/ros2_control.xacro"/>
-  <!-- Base link -->
+  <!-- Base body -->
   <link name="base_link">
     <visual>
       <geometry>
-        <box size="0.5 0.3 0.1"/>
+        <box size="0.457 0.457 0.1"/>
       </geometry>
-      <origin xyz="0 0 0.25"/>
-      <material name="blue">
-        <color rgba="0 0 0.8 1"/>
+      <origin xyz="0 0 0.15"/>
+      <material name="red">
+        <color rgba="0.8 0.0 0.0 1.0"/>
       </material>
     </visual>
     <collision>
       <geometry>
-        <box size="0.1 0.3 0.1"/>
+        <box size="0.35 0.3 0.1"/>
       </geometry>
-      <origin xyz="0 0 0.25"/>
+      <origin xyz="0 0 0.15"/>
     </collision>
     <inertial>
-      <origin xyz="0 0 0.25"/>
-      <mass value="10.0"/>
-      <inertia ixx="0.1" iyy="0.1" izz="0.1" ixy="0.0" ixz="0.0" iyz="0.0"/>
+      <origin xyz="0 0 0.15"/>
+      <mass value="8.0"/>
+      <inertia ixx="0.0842" iyy="0.1117" izz="0.1867"
+               ixy="0.0" ixz="0.0" iyz="0.0"/>
     </inertial>
   </link>
-  <!-- Rear Wheels (driven) -->
-  <xacro:wheel_macro prefix="left_rear" parent="base_link" xyz="-0.2 0.19 0.15" friction="1.5"/>
-  <xacro:wheel_macro prefix="right_rear" parent="base_link" xyz="-0.2 -0.19 0.15" friction="1.5"/>
-  <!-- Front Wheels (passive/caster) -->
-  <xacro:wheel_macro prefix="left_front" parent="base_link" xyz="0.2 0.19 0.15" friction="0.05"/>
-  <xacro:wheel_macro prefix="right_front" parent="base_link" xyz="0.2 -0.19 0.15" friction="0.05"/>
-  <!-- Gazebo friction settings -->
+  <!-- Wheels (rear driven, front passive) -->
+  <xacro:wheel_macro prefix="left_rear"  parent="base_link" xyz="-0.15  0.19  0.05" friction="1.5"/>
+  <xacro:wheel_macro prefix="right_rear" parent="base_link" xyz="-0.15 -0.19  0.05" friction="1.5"/>
+  <xacro:wheel_macro prefix="left_front" parent="base_link" xyz="0.15  0.19  0.05" friction="0.5"/>
+  <xacro:wheel_macro prefix="right_front" parent="base_link" xyz="0.15 -0.19  0.05" friction="0.5"/>
+  <!-- Gazebo friction + color -->
   <gazebo reference="base_link">
-    <mu1>0.01</mu1>
-    <mu2>0.01</mu2>
-    <material>Gazebo/Blue</material>
-  </gazebo>
-  <!-- Gazebo plugin (keep this exactly) -->
-  <gazebo>
-    <plugin name="gazebo_ros2_control" filename="libgazebo_ros2_control.so">
-      <parameters>$(find my_rover)/config/rover_controllers.yaml</parameters>
-    </plugin>
+    <mu1>0.2</mu1>
+    <mu2>0.2</mu2>
+    <material>Gazebo/Red</material>
   </gazebo>
 </robot>

File: src/my_rover/urdf/wheel_macro.xacro (robot description, xacro)
@@ -1,25 +1,27 @@
 <?xml version="1.0"?>
-<robot xmlns:xacro="http://www.ros.org/wiki/xacro">
-  <xacro:macro name="wheel_macro" params="prefix parent xyz friction:=1.5">
+<robot xmlns:xacro="http://ros.org/wiki/xacro">
+  <!-- Wheel macro -->
+  <xacro:macro name="wheel_macro" params="prefix parent xyz friction">
     <link name="${prefix}_wheel_link">
       <visual>
         <geometry>
-          <cylinder radius="0.15" length="0.04"/>
+          <cylinder radius="0.10" length="0.04"/>
         </geometry>
         <origin rpy="1.5708 0 0" xyz="0 0 0"/>
         <material name="black">
-          <color rgba="0.2 0.2 0.2 1"/>
+          <color rgba="0 0 0 1"/>
         </material>
       </visual>
       <collision>
         <geometry>
-          <cylinder radius="0.15" length="0.04"/>
+          <cylinder radius="0.10" length="0.04"/>
         </geometry>
         <origin rpy="1.5708 0 0" xyz="0 0 0"/>
       </collision>
       <inertial>
-        <origin rpy="1.5708 0 0" xyz="0 0 0"/>
-        <mass value="2.0"/>
-        <inertia ixx="0.0115" iyy="0.0115" izz="0.0225" ixy="0.0" ixz="0.0" iyz="0.0"/>
+        <mass value="0.5"/>
+        <origin xyz="0 0 0"/>
+        <inertia ixx="0.001" iyy="0.001" izz="0.001"
+                 ixy="0.0" ixz="0.0" iyz="0.0"/>
       </inertial>
     </link>
@@ -27,14 +29,11 @@
       <parent link="${parent}"/>
       <child link="${prefix}_wheel_link"/>
-      <origin xyz="${xyz}"/>
+      <origin xyz="${xyz}" rpy="0 0 0"/>
       <axis xyz="0 1 0"/>
-      <dynamics damping="0.1" friction="0.1"/>
     </joint>
+    <!-- Gazebo wheel properties -->
     <gazebo reference="${prefix}_wheel_link">
       <mu1>${friction}</mu1>
       <mu2>${friction}</mu2>
-      <kp>100000.0</kp>
-      <kd>10.0</kd>
-      <minDepth>0.005</minDepth>
       <material>Gazebo/Black</material>
     </gazebo>
