Commit message: working controllers on mini rover simulation with cmd_vel integration. Rover recieves info from topics and joint_control shows it is working, but not moving visually. Possible friction issue or wheels clipping base

File: src/my_rover/urdf/ros2_control.xacro (robot description, xacro)
@@ -1,18 +1,18 @@
 <?xml version="1.0"?>
 <robot xmlns:xacro="http://www.ros.org/wiki/xacro">
-  <ros2_control name="GazeboSystem" type="system">
-    <hardware>
-      <plugin>gazebo_ros2_control/GazeboSystem</plugin>
-    </hardware>
-    <joint name="left_rear_wheel_joint">
-      <command_interface name="velocity"/>
-      <state_interface name="position"/>
-      <state_interface name="velocity"/>
-    </joint>
-    <joint name="right_rear_wheel_joint">
-      <command_interface name="velocity"/>
-      <state_interface name="position"/>
-      <state_interface name="velocity"/>
-    </joint>
-  </ros2_control>
+    <ros2_control name="GazeboSystem" type="system">
+        <hardware>
+            <plugin>gazebo_ros2_control/GazeboSystem</plugin>
+        </hardware>
+        <joint name="left_rear_wheel_joint">
+            <command_interface name="velocity"/>
+            <state_interface name="position"/>
+            <state_interface name="velocity"/>
+        </joint>
+        <joint name="right_rear_wheel_joint">
+            <command_interface name="velocity"/>
+            <state_interface name="position"/>
+            <state_interface name="velocity"/>
+        </joint>
+    </ros2_control>
 </robot>

File: src/my_rover/urdf/rover.urdf.xacro (robot description, xacro)
@@ -1,7 +1,46 @@
 <?xml version="1.0"?>
-<robot xmlns:xacro="http://www.ros.org/wiki/xacro">
-  <xacro:include filename="$(find my_rover)/urdf/ros2_control.xacro"/>
-  <xacro:include filename="$(find my_rover)/urdf/rover_base.xacro"/>
-  <xacro:ros2_control/>
-  <xacro:rover_base/>
+<robot name="my_rover" xmlns:xacro="http://www.ros.org/wiki/xacro">
+    <xacro:include filename="$(find my_rover)/urdf/wheel_macro.xacro"/>
+    <xacro:include filename="$(find my_rover)/urdf/ros2_control.xacro"/>
+    <!-- Base link -->
+    <link name="base_link">
+        <visual>
+            <geometry>
+                <box size="0.5 0.3 0.1"/>
+            </geometry>
+            <origin xyz="0 0 0.1"/>  <!-- visual location -->
+            <material name="blue">
+                <color rgba="0 0 0.8 1"/>
+            </material>
+        </visual>
+        <collision>
+            <geometry>
+                <box size="0.5 0.3 0.1"/>
+            </geometry>
+            <origin xyz="0 0 0.1"/>  <!-- collision box -->
+        </collision>
+        <inertial>
+            <origin xyz="0 0 0.1"/>  <!-- center of mass -->
+            <mass value="10.0"/>
+            <inertia ixx="0.1" iyy="0.1" izz="0.1" ixy="0.0" ixz="0.0" iyz="0.0"/>
+        </inertial>
+    </link>
+    <!-- Rear Wheels (driven) - at ground level (z=0) -->
+    <xacro:wheel_macro prefix="left_rear" parent="base_link" xyz="-0.2 0.17 0"/>
+    <xacro:wheel_macro prefix="right_rear" parent="base_link" xyz="-0.2 -0.17 0"/>
+    <!-- Front Wheels (passive/caster) -->
+    <xacro:wheel_macro prefix="left_front" parent="base_link" xyz="0.2 0.17 0"/>
+    <xacro:wheel_macro prefix="right_front" parent="base_link" xyz="0.2 -0.17 0"/>
+    <!-- Gazebo friction settings -->
+    <gazebo reference="base_link">
+      <mu1>0.05</mu1>  <!-- TODO FIX THIS -->
+      <mu2>0.05</mu2>
+      <material>Gazebo/Blue</material>
+    </gazebo>
+    <!-- Gazebo plugin -->
+    <gazebo>
+        <plugin name="gazebo_ros2_control" filename="libgazebo_ros2_control.so">
+            <parameters>$(find my_rover)/config/rover_controllers.yaml</parameters>
+        </plugin>
+    </gazebo>
 </robot>

File: src/my_rover/urdf/wheel_macro.xacro (robot description, xacro)
@@ -4,15 +4,25 @@
     <link name="${prefix}_wheel_link">
       <visual>
-        <geometry><cylinder radius="0.05" length="0.02"/></geometry>
+        <geometry><cylinder radius="0.15" length="0.04"/></geometry>
         <origin rpy="1.5708 0 0" xyz="0 0 0"/>
-        <material name="black"/>
+        <material name="black">
+          <color rgba="0.2 0.2 0.2 1"/>
+        </material>
       </visual>
       <collision>
-        <geometry><cylinder radius="0.05" length="0.02"/></geometry>
+        <geometry><cylinder radius="0.15" length="0.04"/></geometry>
         <origin rpy="1.5708 0 0" xyz="0 0 0"/>
+        <surface>
+          <friction>
+            <ode>
+              <mu>1.0</mu>
+              <mu2>1.0</mu2>
+            </ode>
+          </friction>
+        </surface>
       </collision>
       <inertial>
-        <mass value="1.0"/>
-        <inertia ixx="0.01" iyy="0.01" izz="0.01"
+        <mass value="2.0"/>
+        <inertia ixx="0.0115" iyy="0.0115" izz="0.0225"
                  ixy="0.0" ixz="0.0" iyz="0.0"/>
       </inertial>
@@ -24,4 +34,11 @@
       <axis xyz="0 1 0"/>
     </joint>
+    <gazebo reference="${prefix}_wheel_link">
+      <mu1>1.0</mu1>
+      <mu2>1.0</mu2>
+      <kp>1000000.0</kp>
+      <kd>100.0</kd>
+      <material>Gazebo/Black</material>
+    </gazebo>
   </xacro:macro>
 </robot>

Commit message: basic diff drive rover with odom / cmd_vel topics. Can move in gazebo but only with EXTREME FORCE (10k N). Needs fixing

File: src/my_rover/urdf/ros2_control.xacro (robot description, xacro)
@@ -1,18 +1,20 @@
 <?xml version="1.0"?>
 <robot xmlns:xacro="http://www.ros.org/wiki/xacro">
-    <ros2_control name="GazeboSystem" type="system">
-        <hardware>
-            <plugin>gazebo_ros2_control/GazeboSystem</plugin>
-        </hardware>
-        <joint name="left_rear_wheel_joint">
-            <command_interface name="velocity"/>
-            <state_interface name="position"/>
-            <state_interface name="velocity"/>
-        </joint>
-        <joint name="right_rear_wheel_joint">
-            <command_interface name="velocity"/>
-            <state_interface name="position"/>
-            <state_interface name="velocity"/>
-        </joint>
-    </ros2_control>
+  <ros2_control name="GazeboSystem" type="system">
+    <hardware>
+      <plugin>gazebo_ros2_control/GazeboSystem</plugin>
+    </hardware>
+    <!-- Left wheel -->
+    <joint name="left_rear_wheel_joint">
+      <command_interface name="velocity"/>
+      <state_interface name="position"/>
+      <state_interface name="velocity"/>
+    </joint>
+    <!-- Right wheel -->
+    <joint name="right_rear_wheel_joint">
+      <command_interface name="velocity"/>
+      <state_interface name="position"/>
+      <state_interface name="velocity"/>
+    </joint>
+  </ros2_control>
 </robot>

File: src/my_rover/urdf/rover.urdf.xacro (robot description, xacro)
@@ -1,46 +1,47 @@
 <?xml version="1.0"?>
 <robot name="my_rover" xmlns:xacro="http://www.ros.org/wiki/xacro">
-    <xacro:include filename="$(find my_rover)/urdf/wheel_macro.xacro"/>
-    <xacro:include filename="$(find my_rover)/urdf/ros2_control.xacro"/>
-    <!-- Base link -->
-    <link name="base_link">
-        <visual>
-            <geometry>
-                <box size="0.5 0.3 0.1"/>
-            </geometry>
-            <origin xyz="0 0 0.1"/>  <!-- visual location -->
-            <material name="blue">
-                <color rgba="0 0 0.8 1"/>
-            </material>
-        </visual>
-        <collision>
-            <geometry>
-                <box size="0.5 0.3 0.1"/>
-            </geometry>
-            <origin xyz="0 0 0.1"/>  <!-- collision box -->
-        </collision>
-        <inertial>
-            <origin xyz="0 0 0.1"/>  <!-- center of mass -->
-            <mass value="10.0"/>
-            <inertia ixx="0.1" iyy="0.1" izz="0.1" ixy="0.0" ixz="0.0" iyz="0.0"/>
-        </inertial>
-    </link>
-    <!-- Rear Wheels (driven) - at ground level (z=0) -->
-    <xacro:wheel_macro prefix="left_rear" parent="base_link" xyz="-0.2 0.17 0"/>
-    <xacro:wheel_macro prefix="right_rear" parent="base_link" xyz="-0.2 -0.17 0"/>
-    <!-- Front Wheels (passive/caster) -->
-    <xacro:wheel_macro prefix="left_front" parent="base_link" xyz="0.2 0.17 0"/>
-    <xacro:wheel_macro prefix="right_front" parent="base_link" xyz="0.2 -0.17 0"/>
-    <!-- Gazebo friction settings -->
-    <gazebo reference="base_link">
-      <mu1>0.05</mu1>  <!-- TODO FIX THIS -->
-      <mu2>0.05</mu2>
-      <material>Gazebo/Blue</material>
-    </gazebo>
-    <!-- Gazebo plugin -->
-    <gazebo>
-        <plugin name="gazebo_ros2_control" filename="libgazebo_ros2_control.so">
-            <parameters>$(find my_rover)/config/rover_controllers.yaml</parameters>
-        </plugin>
-    </gazebo>
+  <!-- Include macros -->
+  <xacro:include filename="$(find my_rover)/urdf/wheel_macro.xacro"/>
+  <xacro:include filename="$(find my_rover)/urdf/ros2_control.xacro"/>
+  <!-- Base link -->
+  <link name="base_link">
+    <visual>
+      <geometry>
+        <box size="0.5 0.3 0.1"/>
+      </geometry>
+      <origin xyz="0 0 0.25"/>
+      <material name="blue">
+        <color rgba="0 0 0.8 1"/>
+      </material>
+    </visual>
+    <collision>
+      <geometry>
+        <box size="0.1 0.3 0.1"/>
+      </geometry>
+      <origin xyz="0 0 0.25"/>
+    </collision>
+    <inertial>
+      <origin xyz="0 0 0.25"/>
+      <mass value="10.0"/>
+      <inertia ixx="0.1" iyy="0.1" izz="0.1" ixy="0.0" ixz="0.0" iyz="0.0"/>
+    </inertial>
+  </link>
+  <!-- Rear Wheels (driven) -->
+  <xacro:wheel_macro prefix="left_rear" parent="base_link" xyz="-0.2 0.19 0.15" friction="1.5"/>
+  <xacro:wheel_macro prefix="right_rear" parent="base_link" xyz="-0.2 -0.19 0.15" friction="1.5"/>
+  <!-- Front Wheels (passive/caster) -->
+  <xacro:wheel_macro prefix="left_front" parent="base_link" xyz="0.2 0.19 0.15" friction="0.05"/>
+  <xacro:wheel_macro prefix="right_front" parent="base_link" xyz="0.2 -0.19 0.15" friction="0.05"/>
+  <!-- Gazebo friction settings -->
+  <gazebo reference="base_link">
+    <mu1>0.01</mu1>
+    <mu2>0.01</mu2>
+    <material>Gazebo/Blue</material>
+  </gazebo>
+  <!-- Gazebo plugin (keep this exactly) -->
+  <gazebo>
+    <plugin name="gazebo_ros2_control" filename="libgazebo_ros2_control.so">
+      <parameters>$(find my_rover)/config/rover_controllers.yaml</parameters>
+    </plugin>
+  </gazebo>
 </robot>

File: src/my_rover/urdf/wheel_macro.xacro (robot description, xacro)
@@ -1,8 +1,10 @@
 <?xml version="1.0"?>
 <robot xmlns:xacro="http://www.ros.org/wiki/xacro">
-  <xacro:macro name="wheel_macro" params="prefix parent xyz">
+  <xacro:macro name="wheel_macro" params="prefix parent xyz friction:=1.5">
     <link name="${prefix}_wheel_link">
       <visual>
-        <geometry><cylinder radius="0.15" length="0.04"/></geometry>
+        <geometry>
+          <cylinder radius="0.15" length="0.04"/>
+        </geometry>
         <origin rpy="1.5708 0 0" xyz="0 0 0"/>
         <material name="black">
@@ -11,19 +13,13 @@
       </visual>
       <collision>
-        <geometry><cylinder radius="0.15" length="0.04"/></geometry>
+        <geometry>
+          <cylinder radius="0.15" length="0.04"/>
+        </geometry>
         <origin rpy="1.5708 0 0" xyz="0 0 0"/>
-        <surface>
-          <friction>
-            <ode>
-              <mu>1.0</mu>
-              <mu2>1.0</mu2>
-            </ode>
-          </friction>
-        </surface>
       </collision>
       <inertial>
+        <origin rpy="1.5708 0 0" xyz="0 0 0"/>
         <mass value="2.0"/>
-        <inertia ixx="0.0115" iyy="0.0115" izz="0.0225"
-                 ixy="0.0" ixz="0.0" iyz="0.0"/>
+        <inertia ixx="0.0115" iyy="0.0115" izz="0.0225" ixy="0.0" ixz="0.0" iyz="0.0"/>
       </inertial>
     </link>
@@ -33,10 +29,12 @@
       <origin xyz="${xyz}"/>
       <axis xyz="0 1 0"/>
+      <dynamics damping="0.1" friction="0.1"/>
     </joint>
     <gazebo reference="${prefix}_wheel_link">
-      <mu1>1.0</mu1>
-      <mu2>1.0</mu2>
-      <kp>1000000.0</kp>
-      <kd>100.0</kd>
+      <mu1>${friction}</mu1>
+      <mu2>${friction}</mu2>
+      <kp>100000.0</kp>
+      <kd>10.0</kd>
+      <minDepth>0.005</minDepth>
       <material>Gazebo/Black</material>
     </gazebo>

Commit message: spawning controllers (NOTE: causes wheels to 'brake'). Rover seems to recieve cmd_vel but not have meaningful rotations

File: src/my_rover/urdf/ros2_control.xacro (robot description, xacro)
@@ -2,19 +2,38 @@
 <robot xmlns:xacro="http://www.ros.org/wiki/xacro">
   <ros2_control name="GazeboSystem" type="system">
-    <hardware>
-      <plugin>gazebo_ros2_control/GazeboSystem</plugin>
-    </hardware>
-    <!-- Left wheel -->
-    <joint name="left_rear_wheel_joint">
-      <command_interface name="velocity"/>
-      <state_interface name="position"/>
-      <state_interface name="velocity"/>
-    </joint>
-    <!-- Right wheel -->
-    <joint name="right_rear_wheel_joint">
-      <command_interface name="velocity"/>
-      <state_interface name="position"/>
-      <state_interface name="velocity"/>
-    </joint>
-  </ros2_control>
+  <hardware>
+    <plugin>gazebo_ros2_control/GazeboSystem</plugin>
+  </hardware>
+  <joint name="left_rear_wheel_joint">
+    <command_interface name="velocity"/>
+    <state_interface name="position"/>
+    <state_interface name="velocity"/>
+  </joint>
+  <joint name="right_rear_wheel_joint">
+    <command_interface name="velocity"/>
+    <state_interface name="position"/>
+    <state_interface name="velocity"/>
+  </joint>
+</ros2_control>
+<!-- Transmissions (for gazebo_ros2_control) -->
+<transmission name="left_rear_wheel_trans">
+  <type>transmission_interface/SimpleTransmission</type>
+  <joint name="left_rear_wheel_joint">
+    <hardwareInterface>hardware_interface/VelocityCommandInterface</hardwareInterface>
+  </joint>
+  <actuator name="left_rear_motor">
+    <hardwareInterface>hardware_interface/VelocityCommandInterface</hardwareInterface>
+    <mechanicalReduction>1</mechanicalReduction>
+  </actuator>
+</transmission>
+<transmission name="right_rear_wheel_trans">
+  <type>transmission_interface/SimpleTransmission</type>
+  <joint name="right_rear_wheel_joint">
+    <hardwareInterface>hardware_interface/VelocityCommandInterface</hardwareInterface>
+  </joint>
+  <actuator name="right_rear_motor">
+    <hardwareInterface>hardware_interface/VelocityCommandInterface</hardwareInterface>
+    <mechanicalReduction>1</mechanicalReduction>
+  </actuator>
+</transmission>
 </robot>

File: src/my_rover/urdf/rover.urdf.xacro (robot description, xacro)
@@ -6,16 +6,10 @@
   <link name="base_link">
     <visual>
-      <geometry>
-        <box size="0.457 0.457 0.1"/>
-      </geometry>
+      <geometry><box size="0.457 0.457 0.1"/></geometry>
       <origin xyz="0 0 0.15"/>
-      <material name="red">
-        <color rgba="0.8 0.0 0.0 1.0"/>
-      </material>
+      <material name="red"><color rgba="0.8 0.0 0.0 1.0"/></material>
     </visual>
     <collision>
-      <geometry>
-        <box size="0.35 0.3 0.1"/>
-      </geometry>
+      <geometry><box size="0.35 0.3 0.1"/></geometry>
       <origin xyz="0 0 0.15"/>
     </collision>
@@ -27,14 +21,57 @@
     </inertial>
   </link>
-  <!-- Wheels (rear driven, front passive) -->
+  <!-- Wheels -->
   <xacro:wheel_macro prefix="left_rear"  parent="base_link" xyz="-0.15  0.19  0.05" friction="1.5"/>
   <xacro:wheel_macro prefix="right_rear" parent="base_link" xyz="-0.15 -0.19  0.05" friction="1.5"/>
   <xacro:wheel_macro prefix="left_front" parent="base_link" xyz="0.15  0.19  0.05" friction="0.5"/>
   <xacro:wheel_macro prefix="right_front" parent="base_link" xyz="0.15 -0.19  0.05" friction="0.5"/>
-  <!-- Gazebo friction + color -->
   <gazebo reference="base_link">
-    <mu1>0.2</mu1>
-    <mu2>0.2</mu2>
+    <mu1>10.0</mu1><mu2>10.0</mu2>
     <material>Gazebo/Red</material>
   </gazebo>
+  <!-- ROS2 Control -->
+  <ros2_control name="GazeboSystem" type="system">
+    <hardware>
+      <plugin>gazebo_ros2_control/GazeboSystem</plugin>
+    </hardware>
+    <joint name="left_rear_wheel_joint">
+      <command_interface name="velocity"/>
+      <state_interface name="position"/>
+      <state_interface name="velocity"/>
+    </joint>
+    <joint name="right_rear_wheel_joint">
+      <command_interface name="velocity"/>
+      <state_interface name="position"/>
+      <state_interface name="velocity"/>
+    </joint>
+  </ros2_control>
+  <!-- Transmissions -->
+  <transmission name="left_rear_wheel_trans">
+    <type>transmission_interface/SimpleTransmission</type>
+    <joint name="left_rear_wheel_joint">
+      <hardwareInterface>hardware_interface/VelocityCommandInterface</hardwareInterface>
+    </joint>
+    <actuator name="left_rear_motor">
+      <hardwareInterface>hardware_interface/VelocityCommandInterface</hardwareInterface>
+      <mechanicalReduction>1</mechanicalReduction>
+    </actuator>
+  </transmission>
+  <transmission name="right_rear_wheel_trans">
+    <type>transmission_interface/SimpleTransmission</type>
+    <joint name="right_rear_wheel_joint">
+      <hardwareInterface>hardware_interface/VelocityCommandInterface</hardwareInterface>
+    </joint>
+    <actuator name="right_rear_motor">
+      <hardwareInterface>hardware_interface/VelocityCommandInterface</hardwareInterface>
+      <mechanicalReduction>1</mechanicalReduction>
+    </actuator>
+  </transmission>
+  <!-- Gazebo ROS2 Control Plugin -->
+  <gazebo>
+    <plugin name="gazebo_ros2_control" filename="libgazebo_ros2_control.so">
+      <robot_param>robot_description</robot_param>
+      <robot_param_node>robot_state_publisher</robot_param_node>
+      <parameters>$(find my_rover)/config/rover_controllers.yaml</parameters>
+    </plugin>
+  </gazebo>
 </robot>
