Commit message: adding controllers & keyboard input. failure to see movement in simulation

File: src/my_rover/urdf/ros2_control.xacro (robot description, xacro)
@@ -2,38 +2,17 @@
 <robot xmlns:xacro="http://www.ros.org/wiki/xacro">
   <ros2_control name="GazeboSystem" type="system">
-  <hardware>
-    <plugin>gazebo_ros2_control/GazeboSystem</plugin>
-  </hardware>
-  <joint name="left_rear_wheel_joint">
-    <command_interface name="velocity"/>
-    <state_interface name="position"/>
-    <state_interface name="velocity"/>
-  </joint>
-  <joint name="right_rear_wheel_joint">
-    <command_interface name="velocity"/>
-    <state_interface name="position"/>
-    <state_interface name="velocity"/>
-  </joint>
-</ros2_control>
-<!-- Transmissions (for gazebo_ros2_control) -->
-<transmission name="left_rear_wheel_trans">
-  <type>transmission_interface/SimpleTransmission</type>
-  <joint name="left_rear_wheel_joint">
-    <hardwareInterface>hardware_interface/VelocityCommandInterface</hardwareInterface>
-  </joint>
-  <actuator name="left_rear_motor">
-    <hardwareInterface>hardware_interface/VelocityCommandInterface</hardwareInterface>
-    <mechanicalReduction>1</mechanicalReduction>
-  </actuator>
-</transmission>
-<transmission name="right_rear_wheel_trans">
-  <type>transmission_interface/SimpleTransmission</type>
-  <joint name="right_rear_wheel_joint">
-    <hardwareInterface>hardware_interface/VelocityCommandInterface</hardwareInterface>
-  </joint>
-  <actuator name="right_rear_motor">
-    <hardwareInterface>hardware_interface/VelocityCommandInterface</hardwareInterface>
-    <mechanicalReduction>1</mechanicalReduction>
-  </actuator>
-</transmission>
+    <hardware>
+      <plugin>gazebo_ros2_control/GazeboSystem</plugin>
+    </hardware>
+    <joint name="left_rear_wheel_joint">
+      <command_interface name="velocity"/>
+      <state_interface name="position"/>
+      <state_interface name="velocity"/>
+    </joint>
+    <joint name="right_rear_wheel_joint">
+      <command_interface name="velocity"/>
+      <state_interface name="position"/>
+      <state_interface name="velocity"/>
+    </joint>
+  </ros2_control>
 </robot>

File: src/my_rover/urdf/rover.urdf.xacro (robot description, xacro)
@@ -1,5 +1,4 @@
 <?xml version="1.0"?>
 <robot name="rover" xmlns:xacro="http://ros.org/wiki/xacro">
-  <!-- Include wheel macro -->
   <xacro:include filename="$(find my_rover)/urdf/wheel_macro.xacro"/>
   <!-- Base body -->
@@ -8,8 +7,10 @@
       <geometry><box size="0.457 0.457 0.1"/></geometry>
       <origin xyz="0 0 0.15"/>
-      <material name="red"><color rgba="0.8 0.0 0.0 1.0"/></material>
+      <material name="red">
+        <color rgba="0.8 0.0 0.0 1.0"/>
+      </material>
     </visual>
     <collision>
-      <geometry><box size="0.35 0.3 0.1"/></geometry>
+      <geometry><box size="0.457 0.457 0.1"/></geometry>
       <origin xyz="0 0 0.15"/>
     </collision>
@@ -22,10 +23,12 @@
   </link>
   <!-- Wheels -->
-  <xacro:wheel_macro prefix="left_rear"  parent="base_link" xyz="-0.15  0.19  0.05" friction="1.5"/>
-  <xacro:wheel_macro prefix="right_rear" parent="base_link" xyz="-0.15 -0.19  0.05" friction="1.5"/>
-  <xacro:wheel_macro prefix="left_front" parent="base_link" xyz="0.15  0.19  0.05" friction="0.5"/>
-  <xacro:wheel_macro prefix="right_front" parent="base_link" xyz="0.15 -0.19  0.05" friction="0.5"/>
+  <xacro:wheel_macro prefix="left_rear"  parent="base_link" xyz="-0.15  0.19  0.05" friction="10.0"/>
+  <xacro:wheel_macro prefix="right_rear" parent="base_link" xyz="-0.15 -0.19  0.05" friction="10.0"/>
+  <xacro:wheel_macro prefix="left_front" parent="base_link" xyz="0.15  0.19  0.05" friction="1.5"/>
+  <xacro:wheel_macro prefix="right_front" parent="base_link" xyz="0.15 -0.19  0.05" friction="1.5"/>
+  <!-- Gazebo base properties -->
   <gazebo reference="base_link">
-    <mu1>10.0</mu1><mu2>10.0</mu2>
+    <mu1>10.0</mu1>
+    <mu2>10.0</mu2>
     <material>Gazebo/Red</material>
   </gazebo>
@@ -46,25 +49,4 @@
     </joint>
   </ros2_control>
-  <!-- Transmissions -->
-  <transmission name="left_rear_wheel_trans">
-    <type>transmission_interface/SimpleTransmission</type>
-    <joint name="left_rear_wheel_joint">
-      <hardwareInterface>hardware_interface/VelocityCommandInterface</hardwareInterface>
-    </joint>
-    <actuator name="left_rear_motor">
-      <hardwareInterface>hardware_interface/VelocityCommandInterface</hardwareInterface>
-      <mechanicalReduction>1</mechanicalReduction>
-    </actuator>
-  </transmission>
-  <transmission name="right_rear_wheel_trans">
-    <type>transmission_interface/SimpleTransmission</type>
-    <joint name="right_rear_wheel_joint">
-      <hardwareInterface>hardware_interface/VelocityCommandInterface</hardwareInterface>
-    </joint>
-    <actuator name="right_rear_motor">
-      <hardwareInterface>hardware_interface/VelocityCommandInterface</hardwareInterface>
-      <mechanicalReduction>1</mechanicalReduction>
-    </actuator>
-  </transmission>
   <!-- Gazebo ROS2 Control Plugin -->
   <gazebo>

File: src/my_rover/urdf/wheel_macro.xacro (robot description, xacro)
@@ -1,5 +1,4 @@
 <?xml version="1.0"?>
 <robot xmlns:xacro="http://ros.org/wiki/xacro">
-  <!-- Wheel macro -->
   <xacro:macro name="wheel_macro" params="prefix parent xyz friction">
     <link name="${prefix}_wheel_link">
@@ -20,7 +19,7 @@
       </collision>
       <inertial>
-        <mass value="0.5"/>
+        <mass value="2.0"/>
         <origin xyz="0 0 0"/>
-        <inertia ixx="0.001" iyy="0.001" izz="0.001"
+        <inertia ixx="0.01" iyy="0.01" izz="0.01"
                  ixy="0.0" ixz="0.0" iyz="0.0"/>
       </inertial>
@@ -32,5 +31,4 @@
       <axis xyz="0 1 0"/>
     </joint>
-    <!-- Gazebo wheel properties -->
     <gazebo reference="${prefix}_wheel_link">
       <mu1>${friction}</mu1>
